File: IoT_Kicad_MP/IoT_Kicad_MP.kicad_sch (KiCad schematic)
At the start: 17 parts, among them IC1 TPS7A2128PYWDJ, IC2 TMP117AIDRVR, IC3 MCP73831T-2DCI_MC, J1 Conn_batt, P1 USB_C_Plug, U1 ESP32-C3-WROOM-02

Commit message: Fichier schéma + routage
Parts:
- removed P1: USB_C_Plug, symbol Connector:USB_C_Plug
- added D2, D3: Green, LED_SMD:LED_0805_2012Metric, symbol Device:LED
- added J2: USB_C_Receptacle_USB2.0_14P, Connector_USB:USB_C_Receptacle_JAE_DX07S016JA1R1500, symbol Connector:USB_C_Receptacle_USB2.0_14P
- added R5: 5k, Resistor_SMD:R_0805_2012Metric, symbol Device:R
- added R6: 330, Resistor_SMD:R_0805_2012Metric, symbol Device:R
- added S1: 09.10201.02, 091020102, symbol Library_IoT_MP:09.10201.02
- C1, C2, C3, C4: footprint (none) -> Capacitor_SMD:C_0805_2012Metric
- C5: value C -> 4.7uF; footprint (none) -> Capacitor_SMD:C_0805_2012Metric
- C6: value C -> 4.7 uF; footprint (none) -> Capacitor_SMD:C_0805_2012Metric
- D1: value LED -> Red; footprint (none) -> LED_SMD:LED_0805_2012Metric
- J1: footprint (none) -> Connector_Wire:SolderWire-0.1sqmm_1x02_P3.6mm_D0.4mm_OD1mm
- R1, R2, R3, R4: footprint (none) -> Resistor_SMD:R_0805_2012Metric
Connections:
- net +3.3V: now also R5.1, S1.2 (NO)
- net +BATT: now also IC1.B1 (EN)
- net GND: now also IC3.9 (EP), D2.1 (K), D3.1 (K), J2.A1 (GND), J2.A12 (GND), J2.B1 (GND), J2.B12 (GND), J2.S1 (SHIELD)
- net USB_D+: now also J2.A6 (D+), J2.B6 (D+)
- net USB_D-: now also J2.A7 (D-), J2.B7 (D-)
- net at C5.1, D1.2 (A), IC3.1 (VDD_1): now also J2.A4 (VBUS), J2.A9 (VBUS), J2.B4 (VBUS), J2.B9 (VBUS)
- net at IC3.5 (STAT), R4.2: now also D3.2 (A)
- net at IC2.3 (ALERT): now also R5.2
- net at U1.2 (EN): now also D2.2 (A), R6.2
- new net: R6.1, S1.1 (COM)
Other:
- note added: "Alimentation + régulation"
- note added: "Capteur temp."
- note added: "Rechargement + transmission USB + gestion charge batterie"
- note added: "Unité de traitement"
- moved on the sheet: C5, C6, D1, IC3, R1, R4
